File: hackpad.kicad_sch (KiCad schematic)
At the start: 40 parts, among them J1 OLED_Display, SW1 SW_Push, SW10 SW_Push, SW11 SW_Push, SW12 SW_Push, SW13 SW_Push, SW14 SW_Push, SW15 SW_Push, SW16 SW_Push, SW17 SW_Push, SW18 SW_Push, SW19 SW_Push, SW2 SW_Push, SW3 SW_Push, SW4 SW_Push, SW5 SW_Push, SW6 SW_Push, SW7 SW_Push, SW8 SW_Push, SW9 SW_Push, U1 SEEED-XIAO

Commit message: idk
Parts:
- J1: footprint (none) -> e:SSD1306-0.91-OLED-4pin-128x32
- SW1, SW10, SW11, SW12, SW13, SW14, SW15, SW16, SW17, SW18, SW19, SW2, SW3, SW4, SW5, SW6, SW7, SW8, SW9: footprint (none) -> Button_Switch_Keyboard:SW_Cherry_MX_1.00u_PCB
- U1: footprint XIAO_PCB:XIAO-14P-SMD-2.54-21x17.8MM -> Seeeduino-xiao-rp2040-KiCAD-Library:MOUDLE14P-2.54-21X17.8MM
Connections:
- net VCC: now also J1.3 (Pin_3), U1.10 (3V3)
Other:
- moved on the sheet: D1, D10, D11, D12, D13, D14, D15, D16, D17, D18, D19, D2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

Commit message: changed some stuff
Parts:
- removed J1: OLED_Display, e:SSD1306-0.91-OLED-4pin-128x32, symbol Connector:Conn_01x04_Socket
- removed U1: SEEED-XIAO, Seeeduino-xiao-rp2040-KiCAD-Library:MOUDLE14P-2.54-21X17.8MM, symbol SEEED-XIAO:SEEED-XIAO
- added J1: OLED_128x32, .kicad_sym:SSD1306-0.91-OLED-4pin-128x32, symbol ScottoKeebs:OLED_128x32
- added M2: XIAO-RP2040, .kicad_sym:XIAO-RP2040, symbol xiao-rp2040:XIAO-RP2040
- renumbered D11 to D10, D13 to D11, D15 to D12, D10 to D13, D12 to D14, D14 to D15, SW11 to SW10, SW13 to SW11, SW15 to SW12, SW10 to SW13, SW12 to SW14, SW14 to SW15
Connections:
- net GND: now also J1.1 (GND), M2.13 (GND)
- net SCL: now also J1.3 (SCL), M2.1 (D0)
- net SDA: now also J1.4 (SDA), M2.2 (D1)
- net col 1: now also M2.8 (D7)
- net col 2: now also M2.9 (D8)
- net col 3: now also M2.10 (D9)
- net col 4: now also M2.11 (D10)
- net row 1: now also M2.7 (D6)
- net row 2: now also M2.6 (D5)
- net row 3: now also M2.5 (D4)
- net row 4: now also M2.4 (D3)
- net row 5: now also M2.3 (D2)
- new net +3V3: J1.2 (VCC), M2.12 (3V3)
- no-connect marks 0 -> 1
